File: Reference/LilyPad_Buzzer-master/Hardware/SparkFun_LilyPad_Buzzer.brd (EAGLE design)
At the start: 20 x 20 mm, 8 parts

Commit message: v35 ready for initial review
Parts:
- U$1, U$4, U$6, U$7: value SEWTAP-NOHOLE2 -> SEWTAP-NOHOLE"; device LilyPad-Wearables:PETAL-NOHOLE-2SIDE -> LilyPad-Wearables:PETAL-NOHOLE
- U$8, U$9: value SEWTAP6 -> SEWTAP_SMALL; device LilyPad-Wearables:PETAL-SMALL-2SIDE -> LilyPad-Wearables:PETAL-SMALL
