File: Reference/LilyPad_LED_Rainbow-master/Hardware/LilyPad_Rainbow_LED_v02.sch (EAGLE design)
At the start: 30 parts

Commit message: v35 ready for initial review
Parts:
- LED+1, LED+2, LED+3, LED+4, LED+5, LED+6, LED+7, LED-1, LED-2, LED-3, LED-4, LED-5, LED-6, LED-7: value SEWTAP6 -> SEWTAP_SMALL-2SIDE; device LilyPad-Wearables:SEWTAP6 -> LilyPad-Wearables:SEWTAP_SMALL-2SIDE
- LED3: device SparkFun-LED:LED-REDLILYPAD -> SparkFun-LED:LED-RED1206
- LED4: value YELLOW -> Yellow
- R1, R2, R3, R4, R5, R6, R7: device SparkFun-Resistors:150OHM-1/10W-1%(0603) -> SparkFun-Resistors:150OHM-0603-1/10W-1%
Changed lines of the file:
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@@
 <?xml version="1.0" encoding="utf-8"?>
 <!DOCTYPE eagle SYSTEM "eagle.dtd">
-<eagle version="7.5.0">
+<eagle version="7.7.0">
 <drawing>
 <settings>
@@
 <layer number="112" name="tSilk" color="7" fill="1" visible="yes" active="yes"/>
 <layer number="113" name="IDFDebug" color="4" fill="1" visible="yes" active="yes"/>
+<layer number="114" name="Badge_Outline" color="7" fill="1" visible="yes" active="yes"/>
+<layer number="115" name="ReferenceISLANDS" color="7" fill="1" visible="yes" active="yes"/>
 <layer number="116" name="Patch_BOT" color="9" fill="4" visible="yes" active="yes"/>
 <layer number="118" name="Rect_Pads" color="7" fill="1" visible="yes" active="yes"/>
@@
 </classes>
 <parts>
-<part name="LED+1" library="LilyPad-Wearables" deviceset="SEWTAP" device="6" value="SEWTAP6"/>
-<part name="LED-1" library="LilyPad-Wearables" deviceset="SEWTAP" device="6" value="SEWTAP6"/>
-<part name="R1" library="SparkFun-Resistors" deviceset="150OHM-1/10W-1%(0603)" device="" value="150"/>
+<part name="LED+1" library="LilyPad-Wearables" deviceset="SEWTAP" device="_SMALL-2SIDE" value="SEWTAP_SMALL-2SIDE"/>
+<part name="LED-1" library="LilyPad-Wearables" deviceset="SEWTAP" device="_SMALL-2SIDE" value="SEWTAP_SMALL-2SIDE"/>
+<part name="R1" library="SparkFun-Resistors" deviceset="150OHM" device="-0603-1/10W-1%" value="150"/>
 <part name="LED1" library="SparkFun-LED" deviceset="LED-WHITE" device="1206" value="WHITE"/>
-<part name="LED+2" library="LilyPad-Wearables" deviceset="SEWTAP" device="6" value="SEWTAP6"/>
-<part name="LED-2" library="LilyPad-Wearables" deviceset="SEWTAP" device="6" value="SEWTAP6"/>
-<part name="R2" library="SparkFun-Resistors" deviceset="150OHM-1/10W-1%(0603)" device="" value="150"/>
+<part name="LED+2" library="LilyPad-Wearables" deviceset="SEWTAP" device="_SMALL-2SIDE" value="SEWTAP_SMALL-2SIDE"/>
+<part name="LED-2" library="LilyPad-Wearables" deviceset="SEWTAP" device="_SMALL-2SIDE" value="SEWTAP_SMALL-2SIDE"/>
+<part name="R2" library="SparkFun-Resistors" deviceset="150OHM" device="-0603-1/10W-1%" value="150"/>
 <part name="LED2" library="SparkFun-LED" deviceset="LED-PINK" device="1206" value="PINK"/>
-<part name="LED+3" library="LilyPad-Wearables" deviceset="SEWTAP" device="6" value="SEWTAP6"/>
-<part name="LED-3" library="LilyPad-Wearables" deviceset="SEWTAP" device="6" value="SEWTAP6"/>
-<part name="R3" library="SparkFun-Resistors" deviceset="150OHM-1/10W-1%(0603)" device="" value="150"/>
-<part name="LED3" library="SparkFun-LED" deviceset="LED-RED" device="LILYPAD" value="RED"/>
-<part name="LED+4" library="LilyPad-Wearables" deviceset="SEWTAP" device="6" value="SEWTAP6"/>
-<part name="LED-4" library="LilyPad-Wearables" deviceset="SEWTAP" device="6" value="SEWTAP6"/>
-<part name="R4" library="SparkFun-Resistors" deviceset="150OHM-1/10W-1%(0603)" device="" value="150"/>
-<part name="LED4" library="SparkFun-LED" deviceset="LED-YELLOW" device="LILYPAD" value="YELLOW"/>
-<part name="LED+5" library="LilyPad-Wearables" deviceset="SEWTAP" device="6" value="SEWTAP6"/>
-<part name="LED-5" library="LilyPad-Wearables" deviceset="SEWTAP" device="6" value="SEWTAP6"/>
-<part name="R5" library="SparkFun-Resistors" deviceset="150OHM-1/10W-1%(0603)" device="" value="150"/>
+<part name="LED+3" library="LilyPad-Wearables" deviceset="SEWTAP" device="_SMALL-2SIDE" value="SEWTAP_SMALL-2SIDE"/>
+<part name="LED-3" library="LilyPad-Wearables" deviceset="SEWTAP" device="_SMALL-2SIDE" value="SEWTAP_SMALL-2SIDE"/>
+<part name="R3" library="SparkFun-Resistors" deviceset="150OHM" device="-0603-1/10W-1%" value="150"/>
+<part name="LED3" library="SparkFun-LED" deviceset="LED-RED" device="1206" value="RED"/>
+<part name="LED+4" library="LilyPad-Wearables" deviceset="SEWTAP" device="_SMALL-2SIDE" value="SEWTAP_SMALL-2SIDE"/>
+<part name="LED-4" library="LilyPad-Wearables" deviceset="SEWTAP" device="_SMALL-2SIDE" value="SEWTAP_SMALL-2SIDE"/>
+<part name="R4" library="SparkFun-Resistors" deviceset="150OHM" device="-0603-1/10W-1%" value="150"/>
+<part name="LED4" library="SparkFun-LED" deviceset="LED-YELLOW" device="LILYPAD" value="Yellow"/>
+<part name="LED+5" library="LilyPad-Wearables" deviceset="SEWTAP" device="_SMALL-2SIDE" value="SEWTAP_SMALL-2SIDE"/>
+<part name="LED-5" library="LilyPad-Wearables" deviceset="SEWTAP" device="_SMALL-2SIDE" value="SEWTAP_SMALL-2SIDE"/>
+<part name="R5" library="SparkFun-Resistors" deviceset="150OHM" device="-0603-1/10W-1%" value="150"/>
 <part name="LED5" library="SparkFun-LED" deviceset="LED-GREEN" device="LILYPAD" value="GREEN"/>
-<part name="LED+6" library="LilyPad-Wearables" deviceset="SEWTAP" device="6" value="SEWTAP6"/>
-<part name="LED-6" library="LilyPad-Wearables" deviceset="SEWTAP" device="6" value="SEWTAP6"/>
-<part name="R6" library="SparkFun-Resistors" deviceset="150OHM-1/10W-1%(0603)" device="" value="150"/>
+<part name="LED+6" library="LilyPad-Wearables" deviceset="SEWTAP" device="_SMALL-2SIDE" value="SEWTAP_SMALL-2SIDE"/>
+<part name="LED-6" library="LilyPad-Wearables" deviceset="SEWTAP" device="_SMALL-2SIDE" value="SEWTAP_SMALL-2SIDE"/>
+<part name="R6" library="SparkFun-Resistors" deviceset="150OHM" device="-0603-1/10W-1%" value="150"/>
 <part name="LED6" library="SparkFun-LED" deviceset="LED-BLUE" device="1206" value="BLUE"/>
-<part name="LED+7" library="LilyPad-Wearables" deviceset="SEWTAP" device="6" value="SEWTAP6"/>
-<part name="LED-7" library="LilyPad-Wearables" deviceset="SEWTAP" device="6" value="SEWTAP6"/>
-<part name="R7" library="SparkFun-Resistors" deviceset="150OHM-1/10W-1%(0603)" device="" value="150"/>
+<part name="LED+7" library="LilyPad-Wearables" deviceset="SEWTAP" device="_SMALL-2SIDE" value="SEWTAP_SMALL-2SIDE"/>
+<part name="LED-7" library="LilyPad-Wearables" deviceset="SEWTAP" device="_SMALL-2SIDE" value="SEWTAP_SMALL-2SIDE"/>
+<part name="R7" library="SparkFun-Resistors" deviceset="150OHM" device="-0603-1/10W-1%" value="150"/>
 <part name="LED7" library="SparkFun-LED" deviceset="LED-WHITE" device="1206" value="WHITE"/>
 <part name="FRAME1" library="SparkFun-Aesthetics" deviceset="FRAME-LETTER" device=""/>
