File: Hardware/main/main.brd (EAGLE design)
At the start: 109.2 x 80.6 mm, 184 parts, among them J1 SEWTAP_LONG, J10 SEWTAP_LONG, J11 SEWTAP_LONG, J12 SEWTAP_LONG, J13 SEWTAP_LONG, J14 SEWTAP_LONG, J15 AMP FCI 10103594-0001LF, J2 SEWTAP_LONG, J3 SEWTAP_LONG, J4 SEWTAP_LONG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

Commit message: Almost ready for review.  Art has been finalized
Parts:
- removed LOGO3: OSHW-LOGOS, SparkFun-Aesthetics:OSHW-LOGO-S@1
- removed U$47: LILYLOGO_SHORT, newLilypadParts:LILYPAD-WEARABLES_LOGO-LILYPAD
- added JP11, JP14: FIDUCIALUFIDUCIAL, SparkFun:MICRO-FIDUCIAL
- added LOGO4, LOGO5, LOGO6: OSHW-LOGOS, SparkFun-Aesthetics:OSHW-LOGO-S
- added R17: 10k, SparkFun-Resistors:0603
- added S3: (no value), SparkFun-Switches:SWITCH_DPDT_SMD_AYZ0202
- added SLIDEOFF, SLIDEON: SEWTAP_MEDIUM-2SIDE, LilyPad-Wearables:PETAL-MEDIUM-2SIDE
- added U$72, U$73: LILYLOGO_ABR, newLilypadParts:LILYPAD-WEARABLES_LOGO-L
- U$1: value LILYLOGO_LONG -> LILYLOGO_SHORT; device newLilypadParts:LILYPAD-WEARABLES_LOGO-LPA -> newLilypadParts:LILYPAD-WEARABLES_LOGO-LILYPAD
- U$43: value LOGO-LPLP -> LILYLOGO_ABR; device LilyPad-Wearables:LOGO-LILYPAD -> newLilypadParts:LILYPAD-WEARABLES_LOGO-L
- moved LOGO1 65.9 mm to (-16.7, 21.3)
- moved LOGO2 65.9 mm to (-23.3, 24.1)
- moved U$43 25.4 mm to (-41.9, -11.4), turned to 90 degrees
- moved D2 7.62 mm to (11.4, -38.1)
- moved D4 7.62 mm to (-27.9, -38.1)
- moved D8 7.62 mm to (21.6, -38.1)
- moved D9 7.62 mm to (27.9, -38.1)
- moved JP1 7.62 mm to (11.4, -43.2)
- moved JP10 7.62 mm to (21.6, -34.3)
- moved JP22 7.62 mm to (-27.9, -34.3)
- moved JP23 7.62 mm to (-27.9, -43.2)
- moved JP5 7.62 mm to (21.6, -43.2)
- moved JP6 7.62 mm to (27.9, -43.2)
- moved JP7 7.62 mm to (11.4, -34.3)
- moved JP9 7.62 mm to (27.9, -34.3)
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Connections:
- new net SINK1: S3.6
- new net SINK2: S3.3
- new net SW_CM: R17.1, S3.2, S3.5, SLIDEOFF.1
- net D9: now also S3.1, S3.4, SLIDEON.1
- net GND: now also R17.2
Routing:
- net GND: track 377.7 -> 627.9 mm
- net 3.3V: track 218.1 -> 305.1 mm
- net D9: track 90.2 -> 159.3 mm
- net D11: track 55.8 -> 90.0 mm
- net D5: track 83.8 -> 116.6 mm
- net SW_CM: track 0.00 -> 32.4 mm
- net D10: track 51.9 -> 80.4 mm
- net D4: track 100.4 -> 128.6 mm
- net D8: track 107.1 -> 133.3 mm
- net D3: track 72.0 -> 98.0 mm
- net D6: track 71.9 -> 93.7 mm
- net D2: track 91.7 -> 112.1 mm
- net D7: track 94.1 -> 111.8 mm
- net SW_CM1: track 0.00 -> 13.0 mm
- net V_BATT: track 34.8 -> 33.2 mm
- added copper zone on layer 16, net 3.3V
- added copper zone on layer 16, net D10
- added copper zone on layer 16, net D11
- added copper zone on layer 16, net D9
- added copper zone on layer 1, net SINK1
- added copper zone on layer 1, net SINK2
- added copper zone on layer 1, net SW_CM
Other:
- board size 109.2 x 80.6 mm -> 109.2 x 82.5 mm
- board text added: "11/SDA"
- board text added: "A2"
- board text added: "A3"
- board text added: "A4"
- board text added: "A5"
- board text added: "A9"
- board text added: "B"
- board text added: "G"
- board text added: "LilyPad Prototyping Board"
- board text added: "Off"
- board text added: "On"
- board text added: "R"
- board text added: "SCL"
- board text added: "SDA"
- board text added: "Switch"
- board text added: "Y"
- board text added: "sparkfun.com/lilypad"
- board text added: "~10"
- board text added: "~10/SCL"
- board text added: "~A8"
- board text removed: "10/SCL"
- board text removed: "10~"
- board text removed: "2"
- board text removed: "3"
- board text removed: "5"
- board text removed: "6~"
- board text removed: "7~"
- board text removed: "8~"
- board text removed: "9"
- board text removed: "V20"
- board text removed: "sparkfun.com/"
- board text removed: "~11/SDA"
- board text removed: "~8"
