File: Hardware/main/main.sch (EAGLE design)
At the start: 127 parts, among them J1 SEWTAP_LONG, J10 SEWTAP_LONG, J11 SEWTAP_LONG, J12 SEWTAP_LONG, J13 SEWTAP_LONG, J14 SEWTAP_LONG, J15 AMP FCI 10103594-0001LF, J2 SEWTAP_LONG, J3 SEWTAP_LONG, J4 SEWTAP_LONG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

Commit message: Almost ready for review.  Art has been finalized
Parts:
- removed U$47: LILYLOGO_SHORT, newLilypadParts:LILYLOGO_SHORT
- added JP11, JP14: FIDUCIALUFIDUCIAL, SparkFun:FIDUCIALUFIDUCIAL
- added LOGO4, LOGO5, LOGO6: OSHW-LOGOS, SparkFun-Aesthetics:OSHW-LOGOS
- added R17: 10k, SparkFun-Resistors:10KOHM-0603-1/10W-1%
- added S3: (no value), SparkFun-Switches:SWITCH-DPDT-SMD-AYZ0202
- added SLIDEOFF, SLIDEON: SEWTAP_MEDIUM-2SIDE, LilyPad-Wearables:SEWTAP_MEDIUM-2SIDE
- added U$43, U$72, U$73: LILYLOGO_ABR, newLilypadParts:LILYLOGO_ABR
- U$1: value LILYLOGO_LONG -> LILYLOGO_SHORT; device newLilypadParts:LILYLOGO_LONG -> newLilypadParts:LILYLOGO_SHORT
Connections:
- new net SINK1: S3.6
- new net SINK2: S3.3
- new net SW_CM: R17.1, S3.2, S3.5, SLIDEOFF.1
- net D9: now also S3.1, S3.4, SLIDEON.1
- net GND: now also R17.2
Other:
- note added: "Switch"
- moved on the sheet: B1, R24, S4, U3
