File: Hardware/LilyPad_Prototyping_Board.brd (EAGLE design)
At the start: 109.2 x 82.5 mm, 193 parts, among them J1 SEWTAP_LONG, J10 SEWTAP_LONG, J11 SEWTAP_LONG, J12 SEWTAP_LONG, J13 SEWTAP_LONG, J14 SEWTAP_LONG, J15 AMP FCI 10103594-0001LF, J2 SEWTAP_LONG, J3 SEWTAP_LONG, J4 SEWTAP_LONG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

Commit message: Ready for review
Parts:
- removed U$69: (no value), newLilypadParts:ROUTE_TICKS
- B1: device SparkFun:BUZZER-CCV -> SparkFun-Electromechanical:BUZZER-CCV
- moved FRAME2 98.2 mm to (-50.8, -68.6)
Routing:
- net GND: track 627.9 -> 637.2 mm
- net D9: track 159.3 -> 168.4 mm
- net 3.3V: track 305.1 -> 312.5 mm
- net D3: track 98.0 -> 102.1 mm
- net D6: track 93.7 -> 96.5 mm
- net D8: track 133.3 -> 136.1 mm
- net D5: track 116.6 -> 119.4 mm
- net D4: track 128.6 -> 131.4 mm
- net D7: track 111.8 -> 114.6 mm
- net D11: track 90.0 -> 92.3 mm
- net D2: track 112.1 -> 114.4 mm
- net D10: track 80.4 -> 82.7 mm
Other:
- board text removed: "All Units Inches"
