File: Hardware/LilyPad_Prototyping_Board.brd (EAGLE design)
At the start: 109.2 x 82.5 mm, 196 parts, among them J1 SEWTAP_LONG-2SIDE, J10 SEWTAP_LONG-2SIDE, J11 SEWTAP_LONG-2SIDE, J12 SEWTAP_LONG-2SIDE, J13 SEWTAP_LONG-2SIDE, J14 SEWTAP_LONG-2SIDE, J15 AMP FCI 10103594-0001LF, J2 SEWTAP_LONG-2SIDE, J3 SEWTAP_LONG-2SIDE, J4 SEWTAP_LONG-2SIDE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

Commit message: Imported new silk
Replaced name and major labeling with polygons derived from Trebuchet
font (LilyPad standard). Polarity and internal labeling left in Eagle
vector font.
Parts:
- added U$43: LILYLOGO_SHORT, newLilypadParts:LILYPAD-WEARABLES_LOGO-LILYPAD
Other:
- board text removed: "11/SDA"
- board text removed: "B"
- board text removed: "G"
- board text removed: "LEDs"
- board text removed: "LilyPad Prototyping Board"
- board text removed: "R"
- board text removed: "USB Plus"
- board text removed: "Y"
- board text removed: "sparkfun.com/lilypad"
- board text removed: "~10/SCL"
