File: Hardware/LilyPad_Prototyping_Board.sch (EAGLE design)
At the start: 138 parts, among them J1 SEWTAP_LONG, J10 SEWTAP_LONG, J11 SEWTAP_LONG, J12 SEWTAP_LONG, J13 SEWTAP_LONG, J14 SEWTAP_LONG, J15 AMP FCI 10103594-0001LF, J2 SEWTAP_LONG, J3 SEWTAP_LONG, J4 SEWTAP_LONG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

Commit message: Ready for review
Parts:
- B1: device SparkFun:BUZZERSMD2 -> SparkFun-Electromechanical:BUZZER-SMD
