File: Hardware/LilyPad_ProtoSnap_Plus.brd (EAGLE design)
At the start: 109.2 x 82.5 mm, 197 parts, among them J1 SEWTAP_LONG-2SIDE, J10 SEWTAP_LONG-2SIDE, J11 SEWTAP_LONG-2SIDE, J12 SEWTAP_LONG-2SIDE, J13 SEWTAP_LONG-2SIDE, J14 SEWTAP_LONG-2SIDE, J15 AMP FCI 10103594-0001LF, J2 SEWTAP_LONG-2SIDE, J3 SEWTAP_LONG-2SIDE, J4 SEWTAP_LONG-2SIDE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

Commit message: Fixed spelling error
Other:
- board text added: "LilyPad concept and shapes by: L. Buechley and N. Seidle"
- board text removed: "LilyPad concept and shapes by: L. Buechly and N. Seidle"

Commit message: Changed bargraph resistors to 470 ohm
To reduce brightness of white LED bargraph, changed R8-R13 inclusive
from 22 ohm to 470 ohm 0402 RES-13829 (new part)
Parts:
- R10, R11, R12, R13, R8, R9: value 22 -> 470
Changed lines of the file:
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@@
 <?xml version="1.0" encoding="utf-8"?>
 <!DOCTYPE eagle SYSTEM "eagle.dtd">
-<eagle version="7.7.0">
+<eagle version="7.4.0">
 <drawing>
 <settings>
@@
 <attribute name="VALUE" value="WHITE" x="49.291875" y="52.07" size="1.778" layer="27" rot="R90" display="off"/>
 </element>
-<element name="R8" library="SparkFun-Resistors" package="0402" value="22" x="49.291875" y="49.291875" rot="R270">
-<attribute name="PROD_ID" value="RES-12427" x="49.291875" y="49.291875" size="1.778" layer="27" rot="R270" display="off"/>
-<attribute name="VALUE" value="22" x="49.291875" y="49.291875" size="1.778" layer="27" rot="R270" display="off"/>
+<element name="R8" library="SparkFun-Resistors" package="0402" value="470" x="49.291875" y="49.291875" rot="R270">
+<attribute name="PROD_ID" value="RES-13829" x="49.291875" y="49.291875" size="1.778" layer="27" rot="R270" display="off"/>
+<attribute name="VALUE" value="470" x="49.291875" y="49.291875" size="1.778" layer="27" rot="R270" display="off"/>
 </element>
 <element name="C2" library="SparkFun-Capacitors" package="0402" value="0.1uF" x="58.800996875" y="55.292628125" rot="R180">
@@
 <attribute name="PROD_ID" value="DIO-09004" x="45.24375" y="52.07" size="1.778" layer="27" rot="R90" display="off"/>
 </element>
-<element name="R9" library="SparkFun-Resistors" package="0402" value="22" x="51.990625" y="49.291875" rot="R270">
-<attribute name="PROD_ID" value="RES-12427" x="51.990625" y="49.291875" size="1.778" layer="27" rot="R270" display="off"/>
-<attribute name="VALUE" value="22" x="51.990625" y="49.291875" size="1.778" layer="27" rot="R270" display="off"/>
+<element name="R9" library="SparkFun-Resistors" package="0402" value="470" x="51.990625" y="49.291875" rot="R270">
+<attribute name="PROD_ID" value="RES-13829" x="51.990625" y="49.291875" size="1.778" layer="27" rot="R270" display="off"/>
+<attribute name="VALUE" value="470" x="51.990625" y="49.291875" size="1.778" layer="27" rot="R270" display="off"/>
 </element>
-<element name="R10" library="SparkFun-Resistors" package="0402" value="22" x="50.64125" y="49.291875" rot="R270">
-<attribute name="PROD_ID" value="RES-12427" x="50.64125" y="49.291875" size="1.778" layer="27" rot="R270" display="off"/>
-<attribute name="VALUE" value="22" x="50.64125" y="49.291875" size="1.778" layer="27" rot="R270" display="off"/>
+<element name="R10" library="SparkFun-Resistors" package="0402" value="470" x="50.64125" y="49.291875" rot="R270">
+<attribute name="PROD_ID" value="RES-13829" x="50.64125" y="49.291875" size="1.778" layer="27" rot="R270" display="off"/>
+<attribute name="VALUE" value="470" x="50.64125" y="49.291875" size="1.778" layer="27" rot="R270" display="off"/>
 </element>
-<element name="R11" library="SparkFun-Resistors" package="0402" value="22" x="45.24375" y="49.291875" rot="R270">
-<attribute name="PROD_ID" value="RES-12427" x="45.24375" y="49.291875" size="1.778" layer="27" rot="R270" display="off"/>
-<attribute name="VALUE" value="22" x="45.24375" y="49.291875" size="1.778" layer="27" rot="R270" display="off"/>
+<element name="R11" library="SparkFun-Resistors" package="0402" value="470" x="45.24375" y="49.291875" rot="R270">
+<attribute name="PROD_ID" value="RES-13829" x="45.24375" y="49.291875" size="1.778" layer="27" rot="R270" display="off"/>
+<attribute name="VALUE" value="470" x="45.24375" y="49.291875" size="1.778" layer="27" rot="R270" display="off"/>
 </element>
 <element name="LED8" library="SparkFun-LED" package="LED-0603" value="WHITE" x="47.9425" y="52.07" rot="R90">
 <attribute name="PROD_ID" value="DIO-09004" x="47.9425" y="52.07" size="1.778" layer="27" rot="R90" display="off"/>
 </element>
-<element name="R12" library="SparkFun-Resistors" package="0402" value="22" x="47.9425" y="49.291875" rot="R270">
-<attribute name="PROD_ID" value="RES-12427" x="47.9425" y="49.291875" size="1.778" layer="27" rot="R270" display="off"/>
-<attribute name="VALUE" value="22" x="47.9425" y="49.291875" size="1.778" layer="27" rot="R270" display="off"/>
+<element name="R12" library="SparkFun-Resistors" package="0402" value="470" x="47.9425" y="49.291875" rot="R270">
+<attribute name="PROD_ID" value="RES-13829" x="47.9425" y="49.291875" size="1.778" layer="27" rot="R270" display="off"/>
+<attribute name="VALUE" value="470" x="47.9425" y="49.291875" size="1.778" layer="27" rot="R270" display="off"/>
 </element>
 <element name="LED9" library="SparkFun-LED" package="LED-0603" value="WHITE" x="46.593125" y="52.07" rot="R90">
 <attribute name="PROD_ID" value="DIO-09004" x="46.593125" y="52.07" size="1.778" layer="27" rot="R90" display="off"/>
 </element>
-<element name="R13" library="SparkFun-Resistors" package="0402" value="22" x="46.593125" y="49.291875" rot="R270">
-<attribute name="PROD_ID" value="RES-12427" x="46.593125" y="49.291875" size="1.778" layer="27" rot="R270" display="off"/>
-<attribute name="VALUE" value="22" x="46.593125" y="49.291875" size="1.778" layer="27" rot="R270" display="off"/>
+<element name="R13" library="SparkFun-Resistors" package="0402" value="470" x="46.593125" y="49.291875" rot="R270">
+<attribute name="PROD_ID" value="RES-13829" x="46.593125" y="49.291875" size="1.778" layer="27" rot="R270" display="off"/>
+<attribute name="VALUE" value="470" x="46.593125" y="49.291875" size="1.778" layer="27" rot="R270" display="off"/>
 </element>
 <element name="FRAME1" library="SparkFun-Aesthetics" package="CREATIVE_COMMONS" value="FRAME-LETTER" x="20.704225" y="-11.43"/>
